Commit message: separate macro for kinematics and gz sensor

File: velodyne_description/urdf/VLP-16.urdf.xacro (robot description, xacro)
@@ -2,5 +2,5 @@
 <robot xmlns:xacro="http://www.ros.org/wiki/xacro" name="VLP-16">
   <xacro:property name="M_PI" value="3.1415926535897931" />
-  <xacro:macro name="VLP-16" params="*origin parent:=base_link name:=velodyne tf_prefix:='' topic:=/velodyne_points organize_cloud:=false hz:=10 lasers:=16 samples:=1875 collision_range:=0.3 min_range:=0.9 max_range:=130.0 noise:=0.008 min_angle:=-${M_PI} max_angle:=${M_PI} gpu:=false">
+  <xacro:macro name="VLP-16" params="*origin parent:=base_link name:=velodyne">
     <joint name="${name}_base_mount_joint" type="fixed">
       <xacro:insert_block name="origin" />
@@ -56,97 +56,43 @@
       </collision>
     </link>
+  </xacro:macro>
+  <xacro:macro name="VLP-16-gz-sensor" params="name:=velodyne tf_prefix:='' topic:=/velodyne_points organize_cloud:=false hz:=10 lasers:=16 samples:=1875 collision_range:=0.3 min_range:=0.9 max_range:=130.0 noise:=0.008 min_angle:=-${M_PI} max_angle:=${M_PI} gpu:=false">
     <!-- Gazebo requires the velodyne_gazebo_plugins package -->
     <gazebo reference="${name}">
-      <xacro:if value="${gpu}">
-        <sensor type="gpu_ray" name="${name}-VLP16">
-          <pose>0 0 0 0 0 0</pose>
-          <visualize>false</visualize>
+      <sensor name='${name}_gpu_lidar' type='gpu_lidar'>
+          <gz_frame_id>${name}</gz_frame_id>
+          <pose relative_to='${name}'>0 0 0 0 0 0</pose>
+          <topic>${topic}</topic>
           <update_rate>${hz}</update_rate>
           <ray>
-            <scan>
-              <horizontal>
-                <samples>${samples}</samples>
-                <resolution>1</resolution>
-                <min_angle>${min_angle}</min_angle>
-                <max_angle>${max_angle}</max_angle>
-              </horizontal>
-              <vertical>
-                <samples>${lasers}</samples>
-                <resolution>1</resolution>
-                <min_angle>-${15.0*M_PI/180.0}</min_angle>
-                <max_angle> ${15.0*M_PI/180.0}</max_angle>
-              </vertical>
-            </scan>
-            <range>
-              <min>${collision_range}</min>
-              <max>${max_range+1}</max>
-              <resolution>0.001</resolution>
-            </range>
-            <noise>
-              <type>gaussian</type>
-              <mean>0.0</mean>
-              <stddev>0.0</stddev>
-            </noise>
+              <scan>
+                  <horizontal>
+                      <samples>${samples}</samples>
+                      <resolution>1</resolution>
+                      <min_angle>${min_angle}</min_angle>
+                      <max_angle>${max_angle}</max_angle>
+                  </horizontal>
+                  <vertical>
+                      <samples>${lasers}</samples>
+                      <resolution>1</resolution>
+                      <min_angle>-${15.0*M_PI/180.0}</min_angle>
+                      <max_angle>${15.0*M_PI/180.0}</max_angle>
+                  </vertical>
+              </scan>
+              <range>
+                  <min>${min_range}</min>
+                  <max>${max_range}</max>
+                  <resolution>0.01</resolution>
+              </range>
+              <noise>
+                <type>gaussian</type>
+                <mean>0.0</mean>
+                <stddev>${noide}</stddev>
+              </noise>
           </ray>
-          <plugin name="gazebo_ros_laser_controller" filename="libgazebo_ros_velodyne_laser.so">
-            <ros>
-              <namespace>/${name}</namespace>
-              <remapping>~/out:=${topic}</remapping>
-            </ros>
-            <tf_prefix>${tf_prefix}</tf_prefix>
-            <frame_name>${name}</frame_name>
-            <organize_cloud>${organize_cloud}</organize_cloud>
-            <min_range>${min_range}</min_range>
-            <max_range>${max_range}</max_range>
-            <gaussian_noise>${noise}</gaussian_noise>
-          </plugin>
-        </sensor>
-      </xacro:if>
-      <xacro:unless value="${gpu}">
-        <sensor type="ray" name="${name}-VLP16">
-          <pose>0 0 0 0 0 0</pose>
-          <visualize>false</visualize>
-          <update_rate>${hz}</update_rate>
-          <ray>
-            <scan>
-              <horizontal>
-                <samples>${samples}</samples>
-                <resolution>1</resolution>
-                <min_angle>${min_angle}</min_angle>
-                <max_angle>${max_angle}</max_angle>
-              </horizontal>
-              <vertical>
-                <samples>${lasers}</samples>
-                <resolution>1</resolution>
-                <min_angle>-${15.0*M_PI/180.0}</min_angle>
-                <max_angle> ${15.0*M_PI/180.0}</max_angle>
-              </vertical>
-            </scan>
-            <range>
-              <min>${collision_range}</min>
-              <max>${max_range+1}</max>
-              <resolution>0.001</resolution>
-            </range>
-            <noise>
-              <type>gaussian</type>
-              <mean>0.0</mean>
-              <stddev>0.0</stddev>
-            </noise>
-          </ray>
-          <plugin name="gazebo_ros_laser_controller" filename="libgazebo_ros_velodyne_laser.so">
-            <ros>
-              <namespace>/${name}</namespace>
-              <remapping>~/out:=${topic}</remapping>
-            </ros>
-            <tf_prefix>${tf_prefix}</tf_prefix>
-            <frame_name>${name}</frame_name>
-            <organize_cloud>${organize_cloud}</organize_cloud>
-            <min_range>${min_range}</min_range>
-            <max_range>${max_range}</max_range>
-            <gaussian_noise>${noise}</gaussian_noise>
-          </plugin>
-        </sensor>
-      </xacro:unless>
-    </gazebo>
+          <always_on>1</always_on>
+          <visualize>true</visualize>
+      </sensor>
+  </gazebo>
   </xacro:macro>
 </robot>
